Commit message: Add marvin collision avoidance demo

File: assets/Marvin_M6_S_CCS_696_V4.0/robot_with_ee.urdf (robot description, URDF)
Before this commit: robot robot_with_ee, 31 links, 30 joints
Joints:
- joint LEFT_EE_TO_HAND_MOUNT: origin xyz=0 0 0 rpy=0 0 -1.5707963 -> xyz=0 0 0 rpy=0 0 3.141592653589793
- joint RIGHT_EE_TO_HAND_MOUNT: origin xyz=0 0 0 rpy=0 0 -1.5707963 -> xyz=0 0 0 rpy=0 0 0
